Commit message: Adjust target positioning

File: src/motoman_gp12_support/urdf/gp12_dual_rail_tool.xacro (robot description, xacro)
@@ -55,5 +55,8 @@
         <mesh filename="package://cosmica_resources/meshes/Itokawa_Hayabusa_200k_poly.stl" scale="${target_model_scale} ${target_model_scale} ${target_model_scale}"/>
       </geometry>
-      <origin xyz="0.0 0.0 0.0" rpy="0 0 0"/>
+      <material name="target_grey">
+        <color rgba="0.5 0.5 0.5 1.0"/>
+      </material>
+      <origin xyz="0.0 0.0 0.25" rpy="0 0 0"/>
     </visual>
     <collision>
@@ -68,5 +71,5 @@
     <parent link="group_2/tool0"/>
     <child link="group_2/target"/>
-    <origin xyz="0 0 0.0" rpy="0 0 0"/>  <!-- offset from tool0 -->
+    <origin xyz="0.0 0.0 0.0" rpy="0 0 0"/>  <!-- offset from tool0 -->
   </joint>
 </robot>
