Commit message: Update urdf for dual + tool

File: src/motoman_gp12_support/urdf/gp12_dual.urdf (robot description, URDF)
Before this commit: robot dual_gp12, 19 links, 18 joints
Links:
- added link group_1/flange
- added link group_2/flange
Joints:
- removed joint group_1/joint_6-tool0
- removed joint group_2/joint_6-tool0
- added joint group_1/flange-tool0: type fixed, parent group_1/flange, child group_1/tool0, origin xyz=0 0 0 rpy=3.1415926 -1.570796 0
- added joint group_1/joint_6-flange: type fixed, parent group_1/link_6, child group_1/flange, origin xyz=0.100 0 0 rpy=0 0 0
- added joint group_2/flange-tool0: type fixed, parent group_2/flange, child group_2/tool0, origin xyz=0 0 0 rpy=3.1415926 -1.570796 0
- added joint group_2/joint_6-flange: type fixed, parent group_2/link_6, child group_2/flange, origin xyz=0.100 0 0 rpy=0 0 0
- joint world_to_robot1: origin xyz=0 0 0 rpy=0 0 0 -> xyz=4.0 0 0 rpy=0 0 3.14159
- joint world_to_robot2: origin xyz=0 1.5 0 rpy=0 0 0 -> xyz=0 0 0 rpy=0 0 0

File: src/motoman_gp12_support/urdf/gp12_dual_rail.urdf (robot description, URDF)
Before this commit: robot dual_gp12_rail, 20 links, 19 joints
Links:
- added link group_1/flange
- added link group_2/flange
- link rail: geometry collision box size=4.0 0.5 0.25; visual box size=4.0 0.5 0.25
Joints:
- removed joint group_1/joint_6-tool0
- removed joint group_2/joint_6-tool0
- added joint group_1/flange-tool0: type fixed, parent group_1/flange, child group_1/tool0, origin xyz=0 0 0 rpy=3.1415926 -1.570796 0
- added joint group_1/joint_6-flange: type fixed, parent group_1/link_6, child group_1/flange, origin xyz=0.100 0 0 rpy=0 0 0
- added joint group_2/flange-tool0: type fixed, parent group_2/flange, child group_2/tool0, origin xyz=0 0 0 rpy=3.1415926 -1.570796 0
- added joint group_2/joint_6-flange: type fixed, parent group_2/link_6, child group_2/flange, origin xyz=0.100 0 0 rpy=0 0 0
- joint rail_joint: limit lower=0.0 upper=3.0 effort=1000.0 velocity=1.0 -> lower=-2.0 upper=2.0 effort=1000.0 velocity=1.0; origin (none) -> xyz=0 0 0.25 rpy=0 0 0
- joint world_to_rail: origin xyz=0 0 0 rpy=0 0 0 -> xyz=4.5 0 0 rpy=0 0 3.14159
- joint world_to_robot2: origin xyz=0 1.5 0 rpy=0 0 0 -> xyz=0 0 0 rpy=0 0 0

File: src/motoman_gp12_support/urdf/gp12_dual_rail_tool.xacro (robot description, xacro)
@@ -12,5 +12,7 @@
   <xacro:property name="rail_height" value="0.25"/>
   <xacro:property name="world_to_rail_offset" value="${rail_length+0.5}"/>
-  <xacro:property name="target_model_scale" value="1.0"/>
+  <xacro:property name="target_model_scale" value="0.001"/>
+  <xacro:property name="target_tool0_offset_xyz" value="0.0 0.0 0.0"/>
+  <xacro:property name="target_tool0_offset_rpy" value="0.0 0.0 0.0"/>
   <!-- Rail for Robot 1 -->
   <link name="rail">
@@ -49,27 +51,34 @@
     <origin xyz="0 0 0" rpy="0 0 0"/>
   </joint>
+  <!-- Explicit mount frame for tuning the target pose relative to Robot 2 -->
+  <link name="group_2/target_mount"/>
+  <joint name="group_2/tool0_to_target_mount" type="fixed">
+    <parent link="group_2/tool0"/>
+    <child link="group_2/target_mount"/>
+    <origin xyz="${target_tool0_offset_xyz}" rpy="${target_tool0_offset_rpy}"/>
+  </joint>
   <!-- Target mounted on Robot 2. NOTE TODO: can be moved to external reusable xacro-->
   <link name="group_2/target">
     <visual>
       <geometry>
-        <mesh filename="package://cosmica_resources/meshes/Itokawa_Hayabusa_200k_poly.stl" scale="${target_model_scale} ${target_model_scale} ${target_model_scale}"/>
+        <mesh filename="package://cosmica_resources/meshes/Itokawa_mockup_assembly.stl" scale="${target_model_scale} ${target_model_scale} ${target_model_scale}"/>
       </geometry>
       <material name="target_grey">
         <color rgba="0.5 0.5 0.5 1.0"/>
       </material>
-      <origin xyz="0.0 0.0 0.25" rpy="0 0 0"/>
+      <origin xyz="0.0 0.0 0.0" rpy="0 0 0"/>
     </visual>
     <collision>
       <geometry>
-        <mesh filename="package://cosmica_resources/meshes/Itokawa_Hayabusa_200k_poly.stl" scale="${target_model_scale} ${target_model_scale} ${target_model_scale}"/>
+        <mesh filename="package://cosmica_resources/meshes/Itokawa_mockup_assembly.stl" scale="${target_model_scale} ${target_model_scale} ${target_model_scale}"/>
       </geometry>
       <origin xyz="0.0 0.0 0.0" rpy="0 0 0"/>
     </collision>
   </link>
-<!-- Define joint from tool0 to link target-->
-  <joint name="group_2/tool0_to_target" type="fixed">
-    <parent link="group_2/tool0"/>
+  <!-- Keep the mesh at the origin of target_mount so alignment is controlled in one place -->
+  <joint name="group_2/target_mount_to_target" type="fixed">
+    <parent link="group_2/target_mount"/>
     <child link="group_2/target"/>
-    <origin xyz="0.0 0.0 0.0" rpy="0 0 0"/>  <!-- offset from tool0 -->
+    <origin xyz="0 0 0" rpy="0 0 0"/>
   </joint>
 </robot>
