Commit message: Update yaskawa urdf to add "flange" link

File: src/motoman_gp12_support/urdf/gp12.urdf (robot description, URDF)
Before this commit: robot motoman_gp12, 9 links, 8 joints
Links:
- added link group_1/flange
Joints:
- removed joint group_1/joint_6-tool0
- added joint group_1/flange-tool0: type fixed, parent group_1/flange, child group_1/tool0, origin xyz=0 0 0 rpy=3.1415926 -1.570796 0
- added joint group_1/joint_6-flange: type fixed, parent group_1/link_6, child group_1/flange, origin xyz=0.100 0 0 rpy=0 0 0

File: src/motoman_gp12_support/urdf/gp12_macro.xacro (robot description, xacro)
@@ -95,4 +95,5 @@
         </collision>
     </link>
+    <link name="${prefix}flange"/>
     <link name="${prefix}tool0"/>
     <!-- end of link list -->
@@ -140,7 +141,14 @@
         <limit lower="-7.9412" upper="7.9412" effort="33.30" velocity="12.2143"/>
     </joint>
-    <joint name="${prefix}joint_6-tool0" type="fixed">
-        <origin xyz="0.100 0 0" rpy="3.1415926 -1.570796 0"/>
+    <!-- ROS-Industrial 'flange' frame: attachment point for EEF models -->
+    <joint name="${prefix}joint_6-flange" type="fixed">
+        <origin xyz="0.100 0 0" rpy="0 0 0"/>
         <parent link="${prefix}link_6"/>
+        <child link="${prefix}flange"/>
+    </joint>
+    <!-- ROS-Industrial 'tool0' frame: all-zeros tool frame -->
+    <joint name="${prefix}flange-tool0" type="fixed">
+        <origin xyz="0 0 0" rpy="3.1415926 -1.570796 0"/>
+        <parent link="${prefix}flange"/>
         <child link="${prefix}tool0"/>
     </joint>
