Commit message: Make all urdf and macro (loads from yaml)

File: src/cosmica_resources/urdf/itokawa_target.xacro (robot description, xacro)
@@ -1,13 +1,75 @@
 <?xml version="1.0" ?>
-<!-- gripper_macro.xacro -->
-<xacro:macro name="gripper" params="prefix parent">
-<link name="${prefix}gripper">
-    <visual>...</visual>
-    <collision>...</collision>
-</link>
-<joint name="${prefix}tool0-gripper" type="fixed">
-    <parent link="${parent}"/>
-    <child link="${prefix}gripper"/>
-    <origin xyz="0 0 0.1" rpy="0 0 0"/>
-</joint>
-</xacro:macro>
+<robot xmlns:xacro="http://ros.org/wiki/xacro">
+  <xacro:macro name="itokawa_target" params="
+      link_name
+      mesh_scale_xyz:='0.001 0.001 0.001'
+      material_rgba:='0.5 0.5 0.5 1.0'
+      mesh_origin_xyz:='0 0 0'
+      mesh_origin_rpy:='0 0 0'
+      collision_margin_scale:='1.05'">
+    <!--
+      Simplified collision box derived from the Itokawa STL axis-aligned bounds.
+      Raw STL extents:
+        x: 803.5884509086609
+        y: 436.65048837661743
+        z: 374.6582889556885
+      Raw STL center:
+        x: 405.6076910495758
+        y: 220.36149287223816
+        z: 203.567156791687
+      The collision box follows the STL axis alignment and scales with mesh_scale_xyz.
+    -->
+    <xacro:property name="mesh_scale_tokens" value="${xacro.tokenize(mesh_scale_xyz)}"/>
+    <xacro:property name="mesh_origin_tokens" value="${xacro.tokenize(mesh_origin_xyz)}"/>
+    <xacro:property name="scale_x" value="${float(mesh_scale_tokens[0])}"/>
+    <xacro:property name="scale_y" value="${float(mesh_scale_tokens[1])}"/>
+    <xacro:property name="scale_z" value="${float(mesh_scale_tokens[2])}"/>
+    <xacro:property name="margin_scale" value="${float(collision_margin_scale)}"/>
+    <xacro:property name="origin_x" value="${float(mesh_origin_tokens[0])}"/>
+    <xacro:property name="origin_y" value="${float(mesh_origin_tokens[1])}"/>
+    <xacro:property name="origin_z" value="${float(mesh_origin_tokens[2])}"/>
+    <xacro:property name="stl_size_x" value="803.5884509086609"/>
+    <xacro:property name="stl_size_y" value="436.65048837661743"/>
+    <xacro:property name="stl_size_z" value="374.6582889556885"/>
+    <xacro:property name="stl_center_x" value="405.6076910495758"/>
+    <xacro:property name="stl_center_y" value="220.36149287223816"/>
+    <xacro:property name="stl_center_z" value="203.567156791687"/>
+    <xacro:property name="collision_size_x" value="${stl_size_x * scale_x * margin_scale}"/>
+    <xacro:property name="collision_size_y" value="${stl_size_y * scale_y * margin_scale}"/>
+    <xacro:property name="collision_size_z" value="${stl_size_z * scale_z * margin_scale}"/>
+    <link name="${link_name}">
+      <visual>
+        <geometry>
+          <mesh filename="package://cosmica_resources/meshes/Itokawa_mockup_assembly.stl" scale="${mesh_scale_xyz}"/>
+        </geometry>
+        <origin xyz="${mesh_origin_xyz}" rpy="${mesh_origin_rpy}"/>
+        <material name="${link_name}_material">
+          <color rgba="${material_rgba}"/>
+        </material>
+      </visual>
+      <!-- Full mesh geometry for collision checks (higher fidelity, lower performance) -->
+      <!-- <collision>
+        <geometry>
+          <mesh filename="package://cosmica_resources/meshes/Itokawa_mockup_assembly.stl" scale="${mesh_scale_xyz}"/>
+        </geometry>
+        <origin xyz="${mesh_origin_xyz}" rpy="${mesh_origin_rpy}"/>
+      </collision> -->
+      <!-- Simplified collision geometry for better performance -->
+      <collision>
+        <geometry>
+          <box size="${collision_size_x} ${collision_size_y} ${collision_size_z}"/>
+        </geometry>
+        <origin
+          xyz="${origin_x + stl_center_x * scale_x} ${origin_y + stl_center_y * scale_y} ${origin_z + stl_center_z * scale_z}"
+          rpy="${mesh_origin_rpy}"/>
+      </collision>
+      <!-- Inertial properties todo next -->
+      <!--
+      <inertial>
+        <mass value="10"/>
+        <inertia ixx="1e-3" ixy="0.0" ixz="0.0" iyy="1e-3" iyz="0.0" izz="1e-3"/>
+      </inertial>
+      -->
+    </link>
+  </xacro:macro>
+</robot>

File: src/motoman_gp12_dual_cell_support/urdf/gp12_dual_cell.xacro (robot description, xacro)
@@ -1,9 +1,11 @@
 <?xml version="1.0" ?>
-<robot name="dual_gp12_rail" xmlns:xacro="http://ros.org/wiki/xacro">
+<robot name="gp12_dual_cell" xmlns:xacro="http://ros.org/wiki/xacro">
   <xacro:arg name="config_file" default="$(find motoman_gp12_dual_cell_support)/config/gp12_dual_cell.yaml" />
+  <xacro:arg name="cell_mode" default="rail" />
+  <xacro:arg name="attach_target" default="true" />
   <xacro:include filename="$(find motoman_gp12_dual_cell_support)/urdf/gp12_dual_cell_macro.xacro" />
   <xacro:gp12_dual_cell
     config_file="$(arg config_file)"
-    cell_mode="rail"
-    attach_target="false" />
+    cell_mode="$(arg cell_mode)"
+    attach_target="$(arg attach_target)" />
 </robot>

File: src/motoman_gp12_dual_cell_support/urdf/gp12_dual_rail_tool.xacro (robot description, xacro)
@@ -1,84 +1,9 @@
 <?xml version="1.0" ?>
 <robot name="dual_gp12_rail" xmlns:xacro="http://ros.org/wiki/xacro">
-  <xacro:include filename="$(find motoman_gp12_support)/urdf/gp12_macro.xacro" />
-  <!-- Instantiate both robots -->
-  <xacro:motoman_gp12 prefix="group_1/"/>
-  <xacro:motoman_gp12 prefix="group_2/"/>
-  <!-- World frame -->
-  <link name="world"/>
-  <!-- Rail size and robot 1 position variables -->
-  <xacro:property name="rail_length" value="4.0"/>
-  <xacro:property name="rail_width" value="0.5"/>
-  <xacro:property name="rail_height" value="0.25"/>
-  <xacro:property name="world_to_rail_offset" value="${rail_length+0.5}"/>
-  <xacro:property name="target_model_scale" value="0.001"/>
-  <xacro:property name="target_tool0_offset_xyz" value="0.0 0.0 0.0"/>
-  <xacro:property name="target_tool0_offset_rpy" value="0.0 0.0 0.0"/>
-  <!-- Rail for Robot 1 -->
-  <link name="rail">
-    <visual>
-      <geometry>
-        <box size="${rail_length} ${rail_width} ${rail_height}"/>
-      </geometry>
-      <origin xyz="0.0 0.0 ${rail_height/2}" rpy="0 0 0"/>
-      <material name="rail_grey">
-        <color rgba="0.5 0.5 0.5 0.5"/>
-      </material>
-    </visual>
-    <collision>
-      <geometry>
-        <box size="${rail_length} ${rail_width} ${rail_height}"/>
-      </geometry>
-      <origin xyz="0.0 0.0 ${rail_height/2}" rpy="0 0 0"/>
-    </collision>
-  </link>
-  <joint name="world_to_rail" type="fixed">
-    <parent link="world"/>
-    <child link="rail"/>
-    <origin xyz="${world_to_rail_offset} 0 0" rpy="0 0 3.14159"/>
-  </joint>
-  <joint name="rail_joint" type="prismatic">
-    <parent link="rail"/>
-    <child link="group_1/base_link"/>
-    <origin xyz="0 0 ${rail_height}" rpy="0 0 0"/>
-    <axis xyz="1 0 0"/>
-    <limit lower="${-rail_length/2}" upper="${rail_length/2}" effort="1000.0" velocity="1.0"/>
-  </joint>
-  <!-- Robot 2 at world origin -->
-  <joint name="world_to_robot2" type="fixed">
-    <parent link="world"/>
-    <child link="group_2/base_link"/>
-    <origin xyz="0 0 0" rpy="0 0 0"/>
-  </joint>
-  <!-- Explicit mount frame for tuning the target pose relative to Robot 2 -->
-  <link name="group_2/target_mount"/>
-  <joint name="group_2/tool0_to_target_mount" type="fixed">
-    <parent link="group_2/tool0"/>
-    <child link="group_2/target_mount"/>
-    <origin xyz="${target_tool0_offset_xyz}" rpy="${target_tool0_offset_rpy}"/>
-  </joint>
-  <!-- Target mounted on Robot 2. NOTE TODO: can be moved to external reusable xacro-->
-  <link name="group_2/target">
-    <visual>
-      <geometry>
-        <mesh filename="package://cosmica_resources/meshes/Itokawa_mockup_assembly.stl" scale="${target_model_scale} ${target_model_scale} ${target_model_scale}"/>
-      </geometry>
-      <material name="target_grey">
-        <color rgba="0.5 0.5 0.5 1.0"/>
-      </material>
-      <origin xyz="0.0 0.0 0.0" rpy="0 0 0"/>
-    </visual>
-    <collision>
-      <geometry>
-        <mesh filename="package://cosmica_resources/meshes/Itokawa_mockup_assembly.stl" scale="${target_model_scale} ${target_model_scale} ${target_model_scale}"/>
-      </geometry>
-      <origin xyz="0.0 0.0 0.0" rpy="0 0 0"/>
-    </collision>
-  </link>
-  <!-- Keep the mesh at the origin of target_mount so alignment is controlled in one place -->
-  <joint name="group_2/target_mount_to_target" type="fixed">
-    <parent link="group_2/target_mount"/>
-    <child link="group_2/target"/>
-    <origin xyz="0 0 0" rpy="0 0 0"/>
-  </joint>
+  <xacro:arg name="config_file" default="$(find motoman_gp12_dual_cell_support)/config/gp12_dual_cell.yaml" />
+  <xacro:include filename="$(find motoman_gp12_dual_cell_support)/urdf/gp12_dual_cell_macro.xacro" />
+  <xacro:gp12_dual_cell
+    config_file="$(arg config_file)"
+    cell_mode="rail"
+    attach_target="true" />
 </robot>
